File: Controller/Controller.kicad_pcb (KiCad board)
At the start: 2 copper layers, 151.1 x 80 mm, 69 parts, among them IC1 LMP7715MF, J1 EC, J10 Chlorine Level, J11 ESP32_JTAG, J12 Temp2, J13 J1B1211CCD, J14 Acid Pump, J15 Chlorine Pump, J16 Filtration Pump, J17 Lighting, J18 Relay_Ext, J19 Flood sensor, J2 Display, J3 ORP, J4 PH, J5 Con_Ext, J6 Pressure, J7 Acid Level, J8 VInput, J9 Temp1, K1 ALQ305, K2 ALQ305, K3 ALQ305, K4 ALQ305, K5 ALQ305, U1 Teensy4.1, U2 ESP32-WROOM-32, U3 V7805-1000, U4 V7803-1000, U5 ULN2003A, U6 1026

Commit message: new schematic
Parts:
- removed C2: 1u, Capacitor_SMD:C_0805_2012Metric_Pad1.18x1.45mm_HandSolder
- removed D5: LED, LED_SMD:LED_1206_3216Metric_Pad1.42x1.75mm_HandSolder
- removed R7: 10k, Resistor_SMD:R_0805_2012Metric_Pad1.20x1.40mm_HandSolder
- removed R9: 150, Resistor_SMD:R_0805_2012Metric_Pad1.20x1.40mm_HandSolder
- removed U2: ESP32-WROOM-32, RF_Module:ESP32-WROOM-32
- removed U6: 1026, SamacSys_Parts:1026
- added J20: EXT_I2C, Connector_JST:JST_PH_B5B-PH-K_1x05_P2.00mm_Vertical, F.Cu at (213.8, 67.6)
- added J21: EXT_UART, Connector_JST:JST_PH_B5B-PH-K_1x05_P2.00mm_Vertical, F.Cu at (213.8, 74.2)
- added J22: 1775485-2, snapeda:TE_1775485-2, F.Cu at (-3.81, 50.5)
- J1: value EC -> Probes
- J11: value ESP32_JTAG -> EXT_2; footprint Connector_JST:JST_PH_B5B-PH-K_1x05_P2.00mm_Vertical -> Connector_JST:JST_PH_B4B-PH-K_1x04_P2.00mm_Vertical
- J2: footprint SamacSys_Parts:L77HDE15SD1CH4F -> Connector_IDC:IDC-Header_2x07_P2.54mm_Latch_Horizontal
- J3: value ORP -> ESP32; footprint Connector_JST:JST_PH_B6B-PH-K_1x06_P2.00mm_Vertical -> Connector_PinSocket_2.54mm:PinSocket_2x03_P2.54mm_Vertical
- J4: value PH -> EXT_SPI; footprint Connector_JST:JST_PH_B6B-PH-K_1x06_P2.00mm_Vertical -> Connector_JST:JST_PH_B7B-PH-K_1x07_P2.00mm_Vertical
- J5: value Con_Ext -> EXT_1; footprint Connector_PinSocket_2.54mm:PinSocket_2x13_P2.54mm_Vertical -> Connector_JST:JST_PH_B5B-PH-K_1x05_P2.00mm_Vertical
- moved J5 136.9 mm to (231.8, 61.1), turned to 0 degrees
- moved J1 74.7 mm to (238.0, 98.8)
- moved J11 66.2 mm to (227.8, 67.6), turned to 0 degrees
- moved J3 44.0 mm to (215.7, 80.3), turned to 0 degrees
- moved J4 41.8 mm to (213.8, 61.1), turned to 0 degrees
- moved J2 27.0 mm to (62.7, 121.9), turned to 270 degrees
Connections:
- J1 pad 4: PH_ORP_SCL -> Probe_SCL
- J1 pad 5: PH_ORP_SDA -> Probe_SDA
- J1 pad 6: EC_PDIS -> Probe_RST
- J11 pad 1: Net-(J11-Pad1) -> GND
- J11 pad 2: Net-(J11-Pad2) -> +3V3
- J11 pad 3: Net-(J11-Pad3) -> EXT_IO3
- J11 pad 4: Net-(J11-Pad4) -> EXT_IO4
- J13 pad 11: Net-(J13-Pad11) -> (no net)
- J13 pad 12: Net-(J13-Pad12) -> (no net)
- J13 pad 13: Net-(J13-Pad13) -> (no net)
- J13 pad 14: Net-(J13-Pad14) -> (no net)
- J13 pad 7: Net-(J13-Pad7) -> (no net)
- J2 pad 10: DISP_RST -> LCD_MOSI
- J2 pad 11: LCD_MOSI -> TOUCH_INT
- J2 pad 12: LCD_SCLK -> LCD_MISO
- J2 pad 13: LCD_CS -> DISP_RST
- J2 pad 14: +5V -> LCD_SCLK
- J2 pad 2: TOUCH_SDA -> +5V
- J2 pad 3: TOUCH_SCL -> GND
- J2 pad 4: TOUCH_INT -> +3V3
- J2 pad 5: DISP_LED2 -> LCD_BackLight
- J2 pad 6: LCD_DC -> LCD_CS
- J2 pad 7: LCD_BackLight -> TOUCH_SDA
- J2 pad 8: LCD_MISO -> LCD_DC
- J2 pad 9: DISP_LED1 -> TOUCH_SCL
- J3 pad 1: +5V -> GND
- J3 pad 3: GND -> ESP_RX
- J3 pad 4: PH_ORP_SCL -> ESP_TX
- J3 pad 5: PH_ORP_SDA -> ESP_BOOT
- J3 pad 6: ORP_PDIS -> ESP_EN
- J4 pad 1: +5V -> GND
- J4 pad 3: GND -> +5V
- J4 pad 4: PH_ORP_SCL -> EXT_SCK
- J4 pad 5: PH_ORP_SDA -> EXT_MOSI
- J4 pad 6: PH_PDIS -> EXT_MISO
- J5 pad 1: +5V -> GND
- J5 pad 2: +5V -> +3V3
- J5 pad 3: EXT_IO4 -> +5V
- J5 pad 4: +3V3 -> EXT_IO1
- U1 pad 15: Net-(U1-Pad15) -> (no net)
- U1 pad 31: EC_PDIS -> (no net)
- U1 pad 32: ORP_PDIS -> (no net)
- U1 pad 33: PH_PDIS -> Probe_RST
- U1 pad 38: PH_ORP_SCL -> Probe_SCL
- U1 pad 39: PH_ORP_SDA -> Probe_SDA
- U1 pad 46: Net-(U1-Pad46) -> (no net)
- U1 pad 49: Net-(U1-Pad49) -> (no net)
- U1 pad 51: Net-(U1-Pad51) -> (no net)
- U1 pad 53: Net-(U1-Pad53) -> (no net)
- U1 pad 54: Net-(U1-Pad54) -> (no net)
- U1 pad 55: Net-(U1-Pad55) -> (no net)
- U1 pad 56: Net-(U1-Pad56) -> (no net)
- U1 pad 57: Net-(U1-Pad57) -> (no net)
- U1 pad 58: Net-(U1-Pad58) -> (no net)
- U1 pad 59: Net-(U1-Pad59) -> (no net)
- U1 pad 66: Net-(U1-Pad66) -> (no net)
- U1 pad 67: Net-(U1-Pad67) -> (no net)
- U1 pad 7: DISP_LED1 -> (no net)
- U1 pad 8: DISP_LED2 -> (no net)
- U5 pad 10: Net-(U5-Pad10) -> (no net)
- U5 pad 11: Net-(U5-Pad11) -> (no net)
- U5 pad 6: Net-(U5-Pad6) -> (no net)
- U5 pad 7: Net-(U5-Pad7) -> (no net)
Routing:
- net GND: track 392.3 -> 77.8 mm, vias 4 -> 0
- net +3V3: track 257.8 -> 3.14 mm, vias 1 -> 0
- net +5V: track 298.3 -> 108.3 mm, vias 1 -> 0
- net PH_ORP_SCL: track 180.9 -> 0.00 mm, vias 1 -> 0
- net PH_ORP_SDA: track 174.9 -> 0.00 mm, vias 1 -> 0
- net EC_PDIS: track 130.9 -> 0.00 mm, vias 1 -> 0
- net PH_PDIS: track 108.6 -> 0.00 mm
- net ORP_PDIS: track 102.4 -> 0.00 mm
- net ESP_BOOT: track 90.3 -> 0.00 mm
- net CHLORINE_LEVEL: track 89.5 -> 0.00 mm
- net ESP_EN: track 89.2 -> 0.00 mm
- net ACID_LEVEL: track 79.1 -> 0.00 mm
- net Net-(J22-Pad1): track 74.3 -> 0.00 mm
- net ESP_TX: track 74.1 -> 0.00 mm
- net ESP_RX: track 70.4 -> 0.00 mm
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
Commit message: board
Parts:
- moved J5 200.3 mm to (31.5, 63.0)
- moved J21 183.4 mm to (31.5, 54.9)
- moved J11 182.1 mm to (45.7, 63.0)
- moved J4 103.7 mm to (115.8, 95.0)
- moved J20 84.0 mm to (134.4, 95.0)
- moved J1 69.2 mm to (172.2, 77.5), turned to 90 degrees
- moved J3 64.8 mm to (151.1, 74.9), turned to 90 degrees
- moved J22 54.8 mm to (50.5, 43.7), turned to 270 degrees
- moved J2 30.3 mm to (68.8, 92.2)
- moved C14 11.7 mm to (109.5, 95.5), turned to 270 degrees
- moved J13 10.7 mm to (95.2, 100.1)
- moved J12 10.7 mm to (148.3, 101.9)
- moved J19 10.7 mm to (127.3, 101.9)
- moved J7 10.7 mm to (110.0, 101.9)
- moved J9 10.7 mm to (137.7, 101.9)
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Connections:
- J1 pad 4: Probe_SCL -> Probe_RST
- J1 pad 5: Probe_SDA -> Probe_SCL
- J1 pad 6: Probe_RST -> Probe_SDA
- J2 pad 10: LCD_MOSI -> LCD_SCLK
- J2 pad 14: LCD_SCLK -> LCD_CS
- J2 pad 6: LCD_CS -> LCD_MOSI
- J21 pad 4: EXT_TX -> EXT_RX
- J21 pad 5: EXT_RX -> EXT_TX
- J3 pad 3: ESP_RX -> ESP_BOOT
- J3 pad 4: ESP_TX -> ESP_EN
- J3 pad 5: ESP_BOOT -> ESP_RX
- J3 pad 6: ESP_EN -> ESP_TX
- J4 pad 5: EXT_MOSI -> EXT_CS
- J4 pad 6: EXT_MISO -> EXT_MOSI
- J4 pad 7: EXT_CS -> EXT_MISO
- J5 pad 2: +3V3 -> +5V
- J5 pad 3: +5V -> +3V3
Routing:
- net +3V3: track 3.14 -> 288.1 mm, vias 0 -> 2
- net +5V: track 108.3 -> 388.0 mm, vias 0 -> 1
- net Probe_SDA: track 0.00 -> 122.5 mm
- net Probe_SCL: track 0.00 -> 120.6 mm
- net Pressure: track 0.00 -> 117.0 mm
- net Probe_RST: track 0.00 -> 109.0 mm
- net ESP_EN: track 0.00 -> 97.0 mm
- net CHLORINE_LEVEL: track 0.00 -> 94.9 mm
- net ESP_TX: track 0.00 -> 85.5 mm
- net flood: track 0.00 -> 84.5 mm
- net ACID_LEVEL: track 0.00 -> 83.8 mm
- net ESP_RX: track 0.00 -> 76.9 mm
- net EXT_SCL: track 0.00 -> 76.6 mm
- net EXT_SDA: track 0.00 -> 76.0 mm
- net ETH_LED: track 0.00 -> 74.2 mm
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
Commit message: board
Routing:
- net GND: track 93.7 -> 140.5 mm, vias 0 -> 17
- net Net-(J22-Pad1): track 49.0 -> 59.0 mm
- net EXT_RX: track 41.2 -> 44.4 mm
- net ACID_LEVEL: track 83.8 -> 85.6 mm
- net Net-(D6-Pad1): track 36.8 -> 38.2 mm
- net Net-(D7-Pad1): track 27.4 -> 28.6 mm
- net CHLORINE_LEVEL: track 94.9 -> 95.7 mm
- net Probe_RST: track 109.0 -> 108.2 mm
- net EXT_SCK: track 70.3 -> 70.9 mm
- net TOUCH_INT: track 33.8 -> 33.2 mm
- net Net-(D8-Pad1): track 19.0 -> 19.6 mm
- added copper zone on B.Cu, net GND
Other:
- rule trace_min: 0.2 -> 0.25
