File: Controller/Controller.sch (KiCad schematic (older format))
At the start: 65 parts, among them IC1 LMP7715MF, J1 EC, J10 Chlorine Level, J11 ESP32_JTAG, J12 Temp2, J13 J1B1211CCD, J14 Acid Pump, J15 Chlorine Pump, J16 Filtration Pump, J17 Lighting, J18 Relay_Ext, J19 Flood sensor, J2 Display, J3 ORP, J4 PH, J5 Con_Ext, J6 Pressure, J7 Acid Level, J8 VInput, J9 Temp1, K1 ALQ305, K2 ALQ305, K3 ALQ305, K4 ALQ305, K5 ALQ305, U1 Teensy4.1, U2 ESP32-WROOM-32, U3 V7805-1000, U4 V7803-1000, U5 ULN2003A, U6 1026

Commit message: new schematic
Parts:
- removed C2: 1u, Capacitor_SMD:C_0805_2012Metric_Pad1.18x1.45mm_HandSolder, symbol Device:C_Small
- removed D5: LED, LED_SMD:LED_1206_3216Metric_Pad1.42x1.75mm_HandSolder, symbol Device:LED
- removed J11: ESP32_JTAG, Connector_JST:JST_PH_B5B-PH-K_1x05_P2.00mm_Vertical, symbol Connector:Conn_01x05_Male
- removed J2: Display, SamacSys_Parts:L77HDE15SD1CH4F, symbol SamacSys_Parts:L77HDE15SD1CH4F
- removed J3: ORP, Connector_JST:JST_PH_B6B-PH-K_1x06_P2.00mm_Vertical, symbol Connector:Conn_01x06_Male
- removed J4: PH, Connector_JST:JST_PH_B6B-PH-K_1x06_P2.00mm_Vertical, symbol Connector:Conn_01x06_Male
- removed J5: Con_Ext, Connector_PinSocket_2.54mm:PinSocket_2x13_P2.54mm_Vertical, symbol Connector_Generic:Conn_02x13_Top_Bottom
- removed R7: 10k, Resistor_SMD:R_0805_2012Metric_Pad1.20x1.40mm_HandSolder, symbol Device:R_Small
- removed R9: 150, Resistor_SMD:R_0805_2012Metric_Pad1.20x1.40mm_HandSolder, symbol Device:R_Small
- removed U2: ESP32-WROOM-32, RF_Module:ESP32-WROOM-32, symbol RF_Module:ESP32-WROOM-32
- removed U6: 1026, SamacSys_Parts:1026, symbol SamacSys_Parts:1026
- added J11: EXT_2, Connector_JST:JST_PH_B4B-PH-K_1x04_P2.00mm_Vertical, symbol Connector_Generic:Conn_01x04
- added J2: Display, Connector_IDC:IDC-Header_2x07_P2.54mm_Latch_Horizontal, symbol Connector_Generic:Conn_02x07_Odd_Even
- added J20: EXT_I2C, Connector_JST:JST_PH_B5B-PH-K_1x05_P2.00mm_Vertical, symbol Connector_Generic:Conn_01x05
- added J21: EXT_UART, Connector_JST:JST_PH_B5B-PH-K_1x05_P2.00mm_Vertical, symbol Connector_Generic:Conn_01x05
- added J22: 1775485-2, TE_1775485-2, symbol 1775485-2:1775485-2
- added J3: ESP32, Connector_PinSocket_2.54mm:PinSocket_2x03_P2.54mm_Vertical, symbol Connector_Generic:Conn_02x03_Odd_Even
- added J4: EXT_SPI, Connector_JST:JST_PH_B7B-PH-K_1x07_P2.00mm_Vertical, symbol Connector_Generic:Conn_01x07
- added J5: EXT_1, Connector_JST:JST_PH_B5B-PH-K_1x05_P2.00mm_Vertical, symbol Connector_Generic:Conn_01x05
- J1: value EC -> Probes
Connections:
- net +3V3: now also J11.2 (Pin_2), J2.4 (Pin_4), J20.2 (Pin_2), J21.3 (Pin_3), J3.2 (Pin_2), J4.2 (Pin_2), J5.2 (Pin_2)
- net +5V: now also J2.2 (Pin_2), J20.3 (Pin_3), J21.2 (Pin_2), J4.3 (Pin_3), J5.3 (Pin_3)
- net DISP_RST: now also J2.13 (Pin_13)
- net ESP_BOOT: now also J3.5 (Pin_5)
- net ESP_EN: now also J3.6 (Pin_6)
- net ESP_RX: now also J3.3 (Pin_3)
- net ESP_TX: now also J3.4 (Pin_4)
- net EXT_CS: now also J4.7 (Pin_7)
- net EXT_IO1: now also J5.4 (Pin_4)
- net EXT_IO2: now also J5.5 (Pin_5)
- net EXT_IO3: now also J11.3 (Pin_3)
- net EXT_IO4: now also J11.4 (Pin_4)
- net EXT_MISO: now also J4.6 (Pin_6)
- net EXT_MOSI: now also J4.5 (Pin_5)
- net EXT_RX: now also J21.5 (Pin_5)
- net EXT_SCK: now also J4.4 (Pin_4)
- net EXT_SCL: now also J20.4 (Pin_4)
- net EXT_SDA: now also J20.5 (Pin_5)
- net EXT_TX: now also J21.4 (Pin_4)
- net GND: now also J11.1 (Pin_1), J2.1 (Pin_1), J2.3 (Pin_3), J20.1 (Pin_1), J21.1 (Pin_1), J3.1 (Pin_1), J4.1 (Pin_1), J5.1 (Pin_1)
- net LCD_BackLight: now also J2.5 (Pin_5)
- net LCD_CS: now also J2.6 (Pin_6)
- net LCD_DC: now also J2.8 (Pin_8)
- net LCD_MISO: now also J2.12 (Pin_12)
- net LCD_MOSI: now also J2.10 (Pin_10)
- net LCD_SCLK: now also J2.14 (Pin_14)
- net TOUCH_INT: now also J2.11 (Pin_11)
- net TOUCH_SCL: now also J2.9 (Pin_9)
- net TOUCH_SDA: now also J2.7 (Pin_7)
- net at U1.50 (VBAT): now also J22.1, J22.3
- net at U1.52 (GND): now also J22.2
- net DISP_LED1: no longer names the net of U1.7 (5_IN2)
- net DISP_LED2: no longer names the net of U1.8 (6_OUT1D)
- net EC_PDIS: no longer names the net of U1.31 (39_MISO1_OUT1A)
- net EC_PDIS: no longer J1.6 (Pin_6)
- net ORP_PDIS: no longer names the net of U1.32 (40_A16)
- net PH_ORP_SCL renamed Probe_SCL
- net PH_ORP_SDA renamed Probe_SDA
- net PH_PDIS renamed Probe_RST
- net Probe_RST: now also J1.6 (Pin_6)
- no-connect marks 46 -> 26

Commit message: board
Parts:
- J22: footprint TE_1775485-2 -> snapeda:TE_1775485-2
Connections:
- net +3V3: now also J5.3 (Pin_3); no longer J5.2 (Pin_2)
- net +5V: now also J5.2 (Pin_2); no longer J5.3 (Pin_3)
- net ESP_BOOT: now also J3.3 (Pin_3); no longer J3.5 (Pin_5)
- net ESP_EN: now also J3.4 (Pin_4); no longer J3.6 (Pin_6)
- net ESP_RX: now also J3.5 (Pin_5); no longer J3.3 (Pin_3)
- net ESP_TX: now also J3.6 (Pin_6); no longer J3.4 (Pin_4)
- net EXT_CS: now also J4.5 (Pin_5); no longer J4.7 (Pin_7)
- net EXT_MISO: now also J4.7 (Pin_7); no longer J4.6 (Pin_6)
- net EXT_MOSI: now also J4.6 (Pin_6); no longer J4.5 (Pin_5)
- net EXT_RX: now also J21.4 (Pin_4); no longer J21.5 (Pin_5)
- net EXT_TX: now also J21.5 (Pin_5); no longer J21.4 (Pin_4)
- net LCD_CS: now also J2.14 (Pin_14); no longer J2.6 (Pin_6)
- net LCD_MOSI: now also J2.6 (Pin_6); no longer J2.10 (Pin_10)
- net LCD_SCLK: now also J2.10 (Pin_10); no longer J2.14 (Pin_14)
- net Probe_RST: now also J1.4 (Pin_4); no longer J1.6 (Pin_6)
- net Probe_SCL: now also J1.5 (Pin_5); no longer J1.4 (Pin_4)
- net Probe_SDA: now also J1.6 (Pin_6); no longer J1.5 (Pin_5)
Changed lines of the file:
@@
 	1    0    0    1
 $EndComp
+Text GLabel 1050 5700 0    50   Input ~ 0
+Probe_SDA
 Text GLabel 1050 5600 0    50   Input ~ 0
-Probe_SDA
-Text GLabel 1050 5500 0    50   Input ~ 0
 Probe_SCL
 $Comp
@@
 Wire Wire Line
 	1100 5400 1200 5400
-Text GLabel 1050 5700 0    50   Input ~ 0
+Text GLabel 1050 5500 0    50   Input ~ 0
 Probe_RST
 Wire Wire Line
@@
 Wire Wire Line
 	6750 4550 6850 4550
+Text GLabel 2850 5700 0    50   Input ~ 0
+ESP_BOOT
 Text GLabel 2850 5800 0    50   Input ~ 0
-ESP_BOOT
-Text GLabel 3350 5700 2    50   Input ~ 0
-ESP_TX
-Text GLabel 2850 5700 0    50   Input ~ 0
 ESP_RX
-Text GLabel 3350 5800 2    50   Input ~ 0
-ESP_EN
 Wire Wire Line
 	8900 4900 9300 4900
@@
 Text GLabel 6050 2600 0    50   Input ~ 0
 EXT_SCL
-Text GLabel 4500 2800 0    50   Input ~ 0
+Text GLabel 4500 2900 0    50   Input ~ 0
 EXT_MISO
+Text GLabel 6050 3700 0    50   Input ~ 0
+EXT_TX
 Text GLabel 6050 3600 0    50   Input ~ 0
-EXT_TX
-Text GLabel 6050 3700 0    50   Input ~ 0
 EXT_RX
 Text GLabel 4500 2600 0    50   Input ~ 0
 EXT_SCK
-Text GLabel 4500 2900 0    50   Input ~ 0
+Text GLabel 4500 2700 0    50   Input ~ 0
 EXT_CS
 $Comp
@@
 L power:+3.3V #PWR014
 U 1 1 61EBC4BE
-P 4500 3400
-F 0 "#PWR014" H 4500 3250 50  0001 C CNN
-F 1 "+3.3V" V 4515 3528 50  0000 L CNN
-F 2 "" H 4500 3400 50  0001 C CNN
-F 3 "" H 4500 3400 50  0001 C CNN
-	1    4500 3400
+P 4500 3500
+F 0 "#PWR014" H 4500 3350 50  0001 C CNN
+F 1 "+3.3V" V 4515 3628 50  0000 L CNN
+F 2 "" H 4500 3500 50  0001 C CNN
+F 3 "" H 4500 3500 50  0001 C CNN
+	1    4500 3500
 	0    -1   -1   0
 $EndComp
@@
 L power:+5V #PWR012
 U 1 1 61EEF14E
-P 4500 3500
-F 0 "#PWR012" H 4500 3350 50  0001 C CNN
-F 1 "+5V" V 4515 3628 50  0000 L CNN
-F 2 "" H 4500 3500 50  0001 C CNN
-F 3 "" H 4500 3500 50  0001 C CNN
-	1    4500 3500
+P 4500 3400
+F 0 "#PWR012" H 4500 3250 50  0001 C CNN
+F 1 "+5V" V 4515 3528 50  0000 L CNN
+F 2 "" H 4500 3400 50  0001 C CNN
+F 3 "" H 4500 3400 50  0001 C CNN
+	1    4500 3400
 	0    -1   -1   0
 $EndComp
@@
 	0    -1   1    0
 $EndComp
-Text GLabel 4500 2700 0    50   Input ~ 0
+Text GLabel 4500 2800 0    50   Input ~ 0
 EXT_MOSI
 $Comp
@@
 	5700 900  5700 800
 Connection ~ 5700 800
-Text GLabel 1600 6800 2    39   Input ~ 0
+Text GLabel 1600 7200 2    39   Input ~ 0
 LCD_CS
 Text GLabel 1100 7200 0    39   Input ~ 0
@@
 Text GLabel 1100 6800 0    39   Input ~ 0
 LCD_BackLight
-Text GLabel 1600 7000 2    39   Input ~ 0
+Text GLabel 1600 6800 2    39   Input ~ 0
 LCD_MOSI
 Text GLabel 1600 7100 2    39   Input ~ 0
@@
 Text GLabel 1100 7000 0    39   Input ~ 0
 TOUCH_SCL
-Text GLabel 1600 7200 2    39   Input ~ 0
+Text GLabel 1600 7000 2    39   Input ~ 0
 LCD_SCLK
 $Comp
@@
 F 0 "J22" H 2050 4330 50  0000 C CNN
 F 1 "1775485-2" H 2100 4800 50  0000 C CNN
-F 2 "TE_1775485-2" H 2050 4600 50  0001 L BNN
+F 2 "snapeda:TE_1775485-2" H 2050 4600 50  0001 L BNN
 F 3 "" H 2050 4600 50  0001 L BNN
 F 4 "Compliant" H 2050 4600 50  0001 L BNN "EU_RoHS_Compliance"
@@
 Wire Wire Line
 	2250 4500 2250 4600
+Text GLabel 3350 5700 2    50   Input ~ 0
+ESP_EN
+Text GLabel 3350 5800 2    50   Input ~ 0
+ESP_TX
 $EndSCHEMATC

Commit message: bom
Parts:
- C14: Manufacturer (none) -> Vishay; digikey BC1084CT-ND -> (none); digikey_pn (none) -> BC1084CT-ND; farnell_pn (none) -> 2860097; manf Vishay K104K15X7RF5TL2 -> (none); mouser_pn (none) -> 594-K104K15X7RF5TL2; mpn (none) -> K104K15X7RF5TL2
- F2: Manufacturer (none) -> Würth Elektronik; digikey_pn (none) -> 732-11370-ND; farnell_pn (none) -> 2471678; mouser_pn (none) -> 710-696101000002
- IC1: Description CMOS Input Amplifiers -> General Purpose Amplifier 1 Circuit Rail-to-Rail; Height 1.45 -> (none); Manufacturer (none) -> Texas Instruments; Manufacturer_Name Texas Instruments -> (none); Manufacturer_Part_Number LMP7715MF -> (none); Mouser Part Number 926-LMP7715MF -> (none); Mouser Price/Stock https://www.mouser.co.uk/ProductDetail/Texas-Instruments/LM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 -> (none); digikey_pn (none) -> LMP7715MF/NOPBCT-ND; farnell_pn (none) -> 3117215; mouser_pn (none) -> 926-LMP7715MF; mpn (none) -> LMP7715MF
- J1: Manufacturer (none) -> JST Sales America Inc.; digikey_pn (none) -> 455-1708-ND; farnell_pn (none) -> 9492453; mpn (none) -> B6B-PH-K-S
- J10, J7: Manufacturer (none) -> JST Sales America Inc.; digikey_pn (none) -> 455-1719-ND; farnell_pn (none) -> 9491902; mpn (none) -> S2B-PH-K-S
- J11: Manufacturer (none) -> JST Sales America Inc.; digikey_pn (none) -> 455-1706-ND; farnell_pn (none) -> 9492437; mpn (none) -> B4B-PH-K-S
- J12, J19, J6, J9: Manufacturer (none) -> JST Sales America Inc.; digikey_pn (none) -> 455-1720-ND; farnell_pn (none) -> 9491910; mpn (none) -> S3B-PH-K-S
- J13: Manufacturer (none) -> Wiznet Technology; Manufacturer_Name Wiznet Technology -> (none); Manufacturer_Part_Number J1B1211CCD -> (none); Mouser Part Number 950-J1B1211CCD -> (none); Mouser Price/Stock http://www.mouser.com/Search/ProductDetail.aspx?qs=6pHq9bjO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 -> (none); digikey_pn (none) -> 1278-1052-ND; mouser_pn (none) -> 950-J1B1211CCD; mpn (none) -> J1B1211CCD
- J14, J15, J16, J17, J18, J8: Manufacturer (none) -> Phoenix Contact; digikey_pn (none) -> 277-1247-ND; farnell_pn (none) -> 3041440; mouser_pn (none) -> 651-1729128; mpn (none) -> 1729128
- J2: Manufacturer (none) -> 3M; digikey_pn (none) -> MHR14N-ND; farnell_pn (none) -> 9838430; mouser_pn (none) -> 517-N3314-5302RB; mpn (none) -> N3314-5302RB
- J20, J21, J5: Manufacturer (none) -> JST Sales America Inc.; digikey_pn (none) -> 455-1707-ND; farnell_pn (none) -> 9492445; mpn (none) -> B5B-PH-K-S
- J22: Comment 1775485-2 -> (none); EU_RoHS_Compliance Compliant -> (none); Manufacturer (none) -> TE Connectivity AMP Connectors; digikey_pn (none) -> A135230-ND; farnell_pn (none) -> 3164752; mouser_pn (none) -> 571-1775485-2; mpn (none) -> 1775485-2
- J4: Manufacturer (none) -> JST Sales America Inc.; digikey_pn (none) -> 455-1709-ND; farnell_pn (none) -> 9491864; mpn (none) -> B7B-PH-K-S
- K1, K2, K3, K4, K5: Description (none) -> General Purpose Relay SPST-NO (1 Form A) 5VDC Coil; MANUFACTURER Panasonic -> (none); MAXIMUM_PACKAGE_HEIGHT 16 mm -> (none); Manufacturer (none) -> Panasonic; PARTREV 2020.08 -> (none); STANDARD Manufacturer Recommendations -> (none); digikey_pn (none) -> 255-3559-ND; farnell_pn (none) -> 2503676; mouser_pn (none) -> 769-ALQ305; mpn (none) -> ALQ305
- U1: Description (none) -> Teensy 4.1 ARM Cortex-M7; Manufacturer (none) -> PJRC; mouser_pn (none) -> 485-4622
- U3: Category Power Supplies - Board Mount -> (none); DK_Datasheet_Link https://www.cui.com/product/resource/digikeypdf/v78xx-1000.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 -> (none); DK_Detail_Page /product-detail/en/cui-inc/V7805-1000/102-1715-ND/1828608 -> (none); Digi-Key_PN 102-1715-ND -> (none); Family DC DC Converters -> (none); MPN V7805-1000 -> (none); Status Active -> (none); digikey_pn (none) -> 102-1715-ND; mpn (none) -> V7805-1000
- U4: Category Power Supplies - Board Mount -> (none); DK_Datasheet_Link https://www.cui.com/product/resource/digikeypdf/v78xx-1000.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 -> (none); DK_Detail_Page /product-detail/en/cui-inc/V7803-1000/102-1714-ND/1828607 -> (none); Digi-Key_PN 102-1714-ND -> (none); Family DC DC Converters -> (none); MPN V7803-1000 -> (none); Status Active -> (none); digikey_pn (none) -> 102-1714-ND; mpn (none) -> V7803-1000
- U5: Manufacturer (none) -> Texas Instruments; digikey_pn (none) -> 296-36174-5-ND; farnell_pn (none) -> 3125096; mouser_pn (none) -> 595-ULN2003ANE4; mpn (none) -> ULN2003ANE4

Commit message: kibot
Parts:
- U3: Manufacturer CUI Inc. -> CUI Inc.
Changed lines of the file:
@@
 F 5 "V7805-1000" H 7200 1400 60  0001 L CNN "mpn"
 F 6 "DC DC CONVERTER 5V 5W" H 7200 1900 60  0001 L CNN "Description"
-F 7 "CUI Inc." H 7200 2000 60  0001 L CNN "Manufacturer"
+F 7 "CUI Inc. " H 7200 2000 60  0001 L CNN "Manufacturer"
 	1    7000 900
 	1    0    0    -1

Commit message: action
Parts:
- U3: Manufacturer CUI Inc. -> CUI Inc.
Changed lines of the file:
@@
 F 5 "V7805-1000" H 7200 1400 60  0001 L CNN "mpn"
 F 6 "DC DC CONVERTER 5V 5W" H 7200 1900 60  0001 L CNN "Description"
-F 7 "CUI Inc. " H 7200 2000 60  0001 L CNN "Manufacturer"
+F 7 "CUI Inc." H 7200 2000 60  0001 L CNN "Manufacturer"
 	1    7000 900
 	1    0    0    -1
