File: Controller/Controller.sch (KiCad schematic (older format))
At the start: 62 parts, among them IC1 LMP7715MF, J1 Probes, J10 Chlorine Level, J11 EXT_2, J12 Temp2, J13 J1B1211CCD, J14 Acid Pump, J15 Chlorine Pump, J16 Filtration Pump, J17 Lighting, J18 Relay_Ext, J19 Flood sensor, J2 Display, J20 EXT_I2C, J21 EXT_UART, J22 1775485-2, J3 ESP32, J4 EXT_SPI, J5 EXT_1, J6 Pressure, J7 Acid Level, J8 VInput, J9 Temp1, K1 ALQ305, K2 ALQ305, K3 ALQ305, K4 ALQ305, K5 ALQ305, U1 Teensy4.1, U3 V7805-1000, U4 V7803-1000, U5 ULN2003A

Commit message: Archive project
Parts:
- C1, C14: symbol Device:C_Small -> archive:Device_C_Small
- C10, C11, C12, C13, C5, C6, C7, C8, C9: symbol Device:C -> archive:Device_C
- C3, C4: symbol Device:CP -> archive:Device_CP
- D10, D6, D7, D8, D9: symbol Device:LED -> archive:Device_LED
- F1: symbol Device:Polyfuse_Small -> archive:Device_Polyfuse_Small
- F2: symbol Device:Fuse_Small -> archive:Device_Fuse_Small
- IC1: symbol SamacSys_Parts:LMP7715MF -> archive:SamacSys_Parts_LMP7715MF
- J1: symbol Connector:Conn_01x06_Male -> archive:Connector_Conn_01x06_Male
- J10, J7: symbol Connector:Conn_01x02_Male -> archive:Connector_Conn_01x02_Male
- J11: symbol Connector_Generic:Conn_01x04 -> archive:Connector_Generic_Conn_01x04
- J12, J6, J9: symbol Connector:Screw_Terminal_01x03 -> archive:Connector_Screw_Terminal_01x03
- J13: symbol SamacSys_Parts:J1B1211CCD -> archive:SamacSys_Parts_J1B1211CCD
- J14, J15, J16, J17, J18, J8: symbol Connector:Screw_Terminal_01x02 -> archive:Connector_Screw_Terminal_01x02
- J19: symbol Connector:Conn_01x03_Male -> archive:Connector_Conn_01x03_Male
- J2: symbol Connector_Generic:Conn_02x07_Odd_Even -> archive:Connector_Generic_Conn_02x07_Odd_Even
- J20, J21, J5: symbol Connector_Generic:Conn_01x05 -> archive:Connector_Generic_Conn_01x05
- J22: symbol 1775485-2:1775485-2 -> archive:1775485-2_1775485-2
- J3: symbol Connector_Generic:Conn_02x03_Odd_Even -> archive:Connector_Generic_Conn_02x03_Odd_Even
- J4: symbol Connector_Generic:Conn_01x07 -> archive:Connector_Generic_Conn_01x07
- K1, K2, K3, K4, K5: symbol ALQ305:ALQ305 -> archive:ALQ305_ALQ305
- L1, L2: symbol Device:L -> archive:Device_L
- R1, R10, R11, R12, R13, R14, R2, R8: symbol Device:R_Small -> archive:Device_R_Small
- U1: symbol teensy:Teensy4.1 -> archive:teensy_Teensy4.1
- U3: symbol dk_DC-DC-Converters:V7805-1000 -> archive:dk_DC-DC-Converters_V7805-1000
- U4: symbol dk_DC-DC-Converters:V7803-1000 -> archive:dk_DC-DC-Converters_V7803-1000
- U5: symbol Transistor_Array:ULN2003A -> archive:Transistor_Array_ULN2003A

Commit message: TE_1775485 -> keystone 1065
Parts:
- removed J22: 1775485-2, snapeda:TE_1775485-2, symbol archive:1775485-2_1775485-2
- added B1: 1065, snapeda:1065, symbol archive:keystone1065_1065
Connections:
- wire segments 230 -> 227
Changed lines of the file:
@@
 NoConn ~ 10600 1300
 NoConn ~ 2000 4400
-Wire Wire Line
-	1850 4600 1850 4450
 Text Notes 4100 2150 0    50   ~ 0
 Extension
@@
 	-1   0    0    1
 $EndComp
-$Comp
-L archive:power_PWR_FLAG #FLG0103
-U 1 1 6303CFB2
-P 1850 4450
-F 0 "#FLG0103" H 1850 4525 50  0001 C CNN
-F 1 "PWR_FLAG" V 1850 4577 50  0000 L CNN
-F 2 "" H 1850 4450 50  0001 C CNN
-F 3 "~" H 1850 4450 50  0001 C CNN
-	1    1850 4450
-	0    -1   -1   0
-$EndComp
-Connection ~ 1850 4450
-Wire Wire Line
-	1850 4450 1850 4400
 $Comp
 L archive:power_+5V #PWR018
@@
 NoConn ~ 1050 1650
 NoConn ~ 1050 1550
-$Comp
-L archive:1775485-2_1775485-2 J22
-U 1 1 612E45E4
-P 2050 4600
-F 0 "J22" H 2050 4330 50  0000 C CNN
-F 1 "1775485-2" H 2100 4800 50  0000 C CNN
-F 2 "snapeda:TE_1775485-2" H 2050 4600 50  0001 L BNN
-F 3 "https://www.te.com/commerce/DocumentDelivery/DDEController?Action=srchrtrv&DocNm=1775485&DocType=Customer+Drawing&DocLang=English" H 2050 4600 50  0001 L BNN
-F 4 "TE Connectivity AMP Connectors" H 2050 4600 50  0001 C CNN "Manufacturer"
-F 5 "A135230-ND" H 2050 4600 50  0001 C CNN "digikey_pn"
-F 6 "3164752" H 2050 4600 50  0001 C CNN "farnell_pn"
-F 7 "571-1775485-2" H 2050 4600 50  0001 C CNN "mouser_pn"
-F 8 "1775485-2" H 2050 4600 50  0001 C CNN "mpn"
-	1    2050 4600
-	-1   0    0    1
-$EndComp
-Wire Wire Line
-	2150 4400 2150 4500
-Wire Wire Line
-	2150 4500 2250 4500
-Wire Wire Line
-	2250 4500 2250 4600
 Text GLabel 3350 5700 2    50   Input ~ 0
 ESP_EN
 Text GLabel 3350 5800 2    50   Input ~ 0
 ESP_TX
+$Comp
+L archive:keystone1065_1065 B1
+U 1 1 613271E7
+P 1850 4600
+F 0 "B1" H 2000 4448 60  0000 C CNN
+F 1 "1065" H 2000 4342 60  0000 C CNN
+F 2 "snapeda:1065" H 2000 4240 60  0001 C CNN
+F 3 "" H 1850 4600 60  0000 C CNN
+	1    1850 4600
+	1    0    0    -1
+$EndComp
+Wire Wire Line
+	2150 4400 2150 4600
+Wire Wire Line
+	1850 4400 1850 4600
 $EndSCHEMATC

Commit message: make more room for relay
Parts:
- F2: footprint SamacSys_Parts:696101000002 -> lib_divers:Fuse-PTF75_Stelvio
Changed lines of the file:
@@
 F 0 "F2" H 5600 807 50  0000 C CNN
 F 1 "Fuse_Small" H 5600 716 50  0001 C CNN
-F 2 "SamacSys_Parts:696101000002" H 5600 900 50  0001 C CNN
+F 2 "lib_divers:Fuse-PTF75_Stelvio" H 5600 900 50  0001 C CNN
 F 3 "https://www.we-online.de/katalog/datasheet/696101000002.pdf" H 5600 900 50  0001 C CNN
 F 4 "Würth Elektronik" H 5600 900 50  0001 C CNN "Manufacturer"

Commit message: ethernet diff tuning
Parts:
- removed C14: 0.1 uF, Capacitor_THT:C_Disc_D3.8mm_W2.6mm_P2.50mm, symbol archive:Device_C_Small
- removed J13: J1B1211CCD, SamacSys_Parts:J1B1211CCD, symbol archive:SamacSys_Parts_J1B1211CCD
- added C2: 0.1uF, Capacitor_THT:CP_Radial_D5.0mm_P2.50mm, symbol Device:CP1_Small
- added J13: Eth, Connector_PinHeader_2.00mm:PinHeader_2x03_P2.00mm_Vertical, symbol Connector_Generic:Conn_02x03_Odd_Even
- added J22: J1B1211CCD, Connector_RJ:RJ45_Cetus_J1B1211CCD_Horizontal, symbol SamacSys_Parts:J1B1211CCD
Connections:
- net labels added: RX+, RX-, TX+, TX-
- net labels removed: ETH_LED, ETH_RX+, ETH_RX-, ETH_TX+, ETH_TX-
- wire segments 227 -> 231
- no-connect marks 26 -> 32
Changed lines of the file:
@@
 $EndComp
-$Comp
-L archive:SamacSys_Parts_J1B1211CCD J13
-U 1 1 6073F9AF
-P 9700 900
-F 0 "J13" H 10150 1165 50  0000 C CNN
-F 1 "J1B1211CCD" H 10150 1074 50  0000 C CNN
-F 2 "SamacSys_Parts:J1B1211CCD" H 10450 1000 50  0001 L CNN
-F 3 "https://www.wiznet.hk/en/index.php?controller=attachment&id_attachment=2" H 10450 900 50  0001 L CNN
-F 4 "SINGLE RJ45 CONNECTOR MODULE WITH 10/100 BASE-TX MAGNETICS AND LEDS" H 10450 800 50  0001 L CNN "Description"
-F 5 "950-J1B1211CCD" H 10450 600 50  0001 L CNN "mouser_pn"
-F 6 "J1B1211CCD" H 10450 300 50  0001 L CNN "mpn"
-F 7 "Wiznet Technology" H 9700 900 50  0001 C CNN "Manufacturer"
-F 8 "1278-1052-ND" H 9700 900 50  0001 C CNN "digikey_pn"
-	1    9700 900
-	1    0    0    -1
-$EndComp
-Wire Wire Line
-	9700 900  9500 900
-Wire Wire Line
-	9700 1000 9650 1000
-Wire Wire Line
-	9700 1100 9500 1100
-Wire Wire Line
-	9700 1200 9500 1200
-Wire Wire Line
-	9700 1300 9650 1300
-Wire Wire Line
-	9650 1300 9650 1000
-Wire Wire Line
-	10600 1000 10700 1000
-Wire Wire Line
-	9700 1400 9500 1400
-Wire Wire Line
-	9650 1300 9650 1800
-Connection ~ 9650 1300
-Wire Wire Line
-	3250 3500 3350 3500
-Wire Wire Line
-	3250 3700 3350 3700
-Wire Wire Line
-	3250 3800 3350 3800
-Wire Wire Line
-	3250 3900 3350 3900
-Wire Wire Line
-	3250 4000 3350 4000
 $Comp
 L archive:ALQ305_ALQ305 K1
@@
 Wire Wire Line
 	3350 2750 3250 2750
-Text GLabel 3350 4000 2    50   Input ~ 0
-ETH_RX+
-Text GLabel 3350 3900 2    50   Input ~ 0
-ETH_LED
-Text GLabel 3350 3800 2    50   Input ~ 0
-ETH_TX-
-Text GLabel 3350 3700 2    50   Input ~ 0
-ETH_TX+
-Text GLabel 3350 3500 2    50   Input ~ 0
-ETH_RX-
-Text GLabel 10800 1100 2    50   Input ~ 0
-ETH_LED
-Text GLabel 9500 1400 0    50   Input ~ 0
-ETH_RX-
-Text GLabel 9500 1200 0    50   Input ~ 0
-ETH_RX+
-Text GLabel 9500 1100 0    50   Input ~ 0
-ETH_TX-
-Text GLabel 9500 900  0    50   Input ~ 0
-ETH_TX+
-NoConn ~ 10600 1400
-NoConn ~ 10600 1300
 NoConn ~ 2000 4400
 Text Notes 4100 2150 0    50   ~ 0
@@
 $EndComp
 $Comp
-L archive:power_GND #PWR0101
-U 1 1 6309BC0B
-P 3300 3600
-F 0 "#PWR0101" H 3300 3350 50  0001 C CNN
-F 1 "GND" V 3305 3472 50  0000 R CNN
-F 2 "" H 3300 3600 50  0001 C CNN
-F 3 "" H 3300 3600 50  0001 C CNN
-	1    3300 3600
-	0    -1   -1   0
-$EndComp
-Wire Wire Line
-	3250 3600 3300 3600
-$Comp
-L archive:power_GND #PWR0102
-U 1 1 630DA049
-P 10850 1850
-F 0 "#PWR0102" H 10850 1600 50  0001 C CNN
-F 1 "GND" H 10855 1677 50  0000 C CNN
-F 2 "" H 10850 1850 50  0001 C CNN
-F 3 "" H 10850 1850 50  0001 C CNN
-	1    10850 1850
-	1    0    0    -1
-$EndComp
-$Comp
 L archive:power_GND #PWR0103
 U 1 1 631356E2
@@
 	5700 800  5850 800
 Connection ~ 5850 800
-Wire Wire Line
-	9650 1800 10050 1800
-Wire Wire Line
-	10250 1800 10700 1800
-$Comp
-L archive:Device_C_Small C14
-U 1 1 607612B2
-P 10150 1800
-F 0 "C14" V 10379 1800 50  0000 C CNN
-F 1 "0.1 uF" V 10288 1800 50  0000 C CNN
-F 2 "Capacitor_THT:C_Disc_D3.8mm_W2.6mm_P2.50mm" H 10150 1800 50  0001 C CNN
-F 3 "http://www.farnell.com/datasheets/2608733.pdf" H 10150 1800 50  0001 C CNN
-F 4 "Vishay" H 10150 1800 50  0001 C CNN "Manufacturer"
-F 5 "BC1084CT-ND" H 10150 1800 50  0001 C CNN "digikey_pn"
-F 6 "K104K15X7RF5TL2" H 10150 1800 50  0001 C CNN "mpn"
-F 7 "2860097" H 10150 1800 50  0001 C CNN "farnell_pn"
-F 8 "594-K104K15X7RF5TL2" H 10150 1800 50  0001 C CNN "mouser_pn"
-	1    10150 1800
-	0    -1   -1   0
-$EndComp
 $Comp
 L archive:Device_Fuse_Small F2
@@
 	0    1    1    0
 $EndComp
-Wire Wire Line
-	10700 1000 10700 1800
-Wire Wire Line
-	10700 1800 10850 1800
-Wire Wire Line
-	10850 1800 10850 1850
-Connection ~ 10700 1800
-Wire Wire Line
-	10800 1100 10600 1100
-NoConn ~ 10600 1200
-NoConn ~ 10600 1500
-NoConn ~ 9700 1500
-Wire Wire Line
-	10600 900  10700 900
-Wire Wire Line
-	10700 900  10700 1000
-Connection ~ 10700 1000
 NoConn ~ 3250 2650
 NoConn ~ 3250 2550
@@
 Wire Wire Line
 	1850 4400 1850 4600
+NoConn ~ 3250 4000
+NoConn ~ 3250 3900
+NoConn ~ 3250 3800
+NoConn ~ 3250 3700
+NoConn ~ 3250 3600
+NoConn ~ 3250 3500
+$Comp
+L SamacSys_Parts:J1B1211CCD J22
+U 1 1 61700052
+P 10150 850
+F 0 "J22" H 10600 1115 50  0000 C CNN
+F 1 "J1B1211CCD" H 10600 1024 50  0000 C CNN
+F 2 "Connector_RJ:RJ45_Cetus_J1B1211CCD_Horizontal" H 10900 950 50  0001 L CNN
+F 3 "http://wizwiki.net/wiki/lib/exe/fetch.php?media=products:wiz550web:wiz550webds_kr:j1b1211ccd.pdf" H 10900 850 50  0001 L CNN
+F 4 "Modules Accessories RJ-45 w/ Transformer Connector /CETUS" H 10900 750 50  0001 L CNN "Description"
+F 5 "" H 10900 650 50  0001 L CNN "Height"
+F 6 "950-J1B1211CCD" H 10900 550 50  0001 L CNN "Mouser Part Number"
+F 7 "https://www.mouser.co.uk/ProductDetail/WIZnet/J1B1211CCD?qs=6pHq9bjOlanFLUlTDcmBeQ%3D%3D" H 10900 450 50  0001 L CNN "Mouser Price/Stock"
+F 8 "WIZnet Inc" H 10900 350 50  0001 L CNN "Manufacturer_Name"
+F 9 "J1B1211CCD" H 10900 250 50  0001 L CNN "Manufacturer_Part_Number"
+	1    10150 850
+	1    0    0    -1
+$EndComp
+$Comp
+L Connector_Generic:Conn_02x03_Odd_Even J13
+U 1 1 617027FA
+P 9500 1150
+F 0 "J13" H 9550 1350 50  0000 C CNN
+F 1 "Eth" H 9550 1650 50  0001 C CNN
+F 2 "Connector_PinHeader_2.00mm:PinHeader_2x03_P2.00mm_Vertical" H 9500 1150 50  0001 C CNN
+F 3 "~" H 9500 1150 50  0001 C CNN
+	1    9500 1150
+	1    0    0    -1
+$EndComp
+$Comp
+L Device:CP1_Small C2
+U 1 1 6170311C
+P 10000 850
+F 0 "C2" H 10200 900 50  0000 R CNN
+F 1 "0.1uF" H 10250 800 50  0000 R CNN
+F 2 "Capacitor_THT:CP_Radial_D5.0mm_P2.50mm" H 10000 850 50  0001 C CNN
+F 3 "~" H 10000 850 50  0001 C CNN
+	1    10000 850
+	-1   0    0    1
+$EndComp
+Wire Wire Line
+	9300 1050 9300 850
+Wire Wire Line
+	9800 1050 10150 1050
+Wire Wire Line
+	9300 850  10150 850
+Wire Wire Line
+	9300 1150 9200 1150
+Wire Wire Line
+	9200 1150 9200 700
+Wire Wire Line
+	9200 700  10000 700
+Wire Wire Line
+	11150 700  11150 850
+Wire Wire Line
+	11150 850  11050 850
+Wire Wire Line
+	11150 850  11150 950
+Wire Wire Line
+	11150 950  11050 950
+Connection ~ 11150 850
+Wire Wire Line
+	11050 1050 11150 1050
+Wire Wire Line
+	11150 1050 11150 1600
+Wire Wire Line
+	11150 1600 9950 1600
+Wire Wire Line
+	9950 1600 9950 1150
+Wire Wire Line
+	9950 1150 9800 1150
+Wire Wire Line
+	10150 1350 9200 1350
+Wire Wire Line
+	9200 1350 9200 1250
+Wire Wire Line
+	9200 1250 9300 1250
+Wire Wire Line
+	9800 1250 10050 1250
+Wire Wire Line
+	10050 1250 10050 1150
+Wire Wire Line
+	10050 1150 10150 1150
+Wire Wire Line
+	10150 1250 10100 1250
+Wire Wire Line
+	10100 1250 10100 950
+Wire Wire Line
+	10100 950  10150 950
+Wire Wire Line
+	10000 750  10000 700
+Connection ~ 10000 700
+Wire Wire Line
+	10000 700  11150 700
+Wire Wire Line
+	10100 950  10000 950
+Connection ~ 10100 950
+NoConn ~ 10150 1450
+NoConn ~ 11050 1450
+NoConn ~ 11050 1350
+NoConn ~ 11050 1250
+NoConn ~ 11050 1150
+Text Label 9400 850  0    50   ~ 0
+TX+
+Text Label 9850 1050 0    50   ~ 0
+TX-
+Text Label 9800 1350 0    50   ~ 0
+RX-
+Text Label 9800 1250 0    50   ~ 0
+RX+
 $EndSCHEMATC

Commit message: relay ethernet too small
Parts:
- added C14: 4.7uF, Capacitor_SMD:C_0805_2012Metric_Pad1.18x1.45mm_HandSolder, symbol archive:Device_C
- added D1: LED, LED_SMD:LED_1206_3216Metric_Pad1.42x1.75mm_HandSolder, symbol archive:Device_LED
- added J23: Relay_Ext, TerminalBlock_Phoenix:TerminalBlock_Phoenix_MKDS-1,5-2-5.08_1x02_P5.08mm_Horizontal, symbol archive:Connector_Screw_Terminal_01x02
- added K6: ALQ305, snapeda:RELAY_ALQ305, symbol archive:ALQ305_ALQ305
- added R3: 180, Resistor_SMD:R_0805_2012Metric_Pad1.20x1.40mm_HandSolder, symbol archive:Device_R_Small
- J18: value Relay_Ext -> Air
Connections:
- wire segments 231 -> 248
- no-connect marks 32 -> 31
Other:
- moved on the sheet: C10, C11, C12, C13, C9, D10, D6, D7, D8, D9, J14, J15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

Commit message: archive
Parts:
- C2: symbol Device:CP1_Small -> archive:Device_CP1_Small
- J13: symbol Connector_Generic:Conn_02x03_Odd_Even -> archive:Connector_Generic_Conn_02x03_Odd_Even
- J22: symbol SamacSys_Parts:J1B1211CCD -> archive:SamacSys_Parts_J1B1211CCD
Changed lines of the file:
@@
 NoConn ~ 3250 3500
 $Comp
-L SamacSys_Parts:J1B1211CCD J22
+L archive:SamacSys_Parts_J1B1211CCD J22
 U 1 1 61700052
 P 10150 850
@@
 $EndComp
 $Comp
-L Connector_Generic:Conn_02x03_Odd_Even J13
+L archive:Connector_Generic_Conn_02x03_Odd_Even J13
 U 1 1 617027FA
 P 9500 1150
@@
 $EndComp
 $Comp
-L Device:CP1_Small C2
+L archive:Device_CP1_Small C2
 U 1 1 6170311C
 P 10000 850

Commit message: JST to SMT
Parts:
- J10, J7: footprint Connector_JST:JST_PH_S2B-PH-K_1x02_P2.00mm_Horizontal -> Connector_JST:JST_PH_S2B-PH-SM4-TB_1x02-1MP_P2.00mm_Horizontal
- J12, J19, J6, J9: footprint Connector_JST:JST_PH_S3B-PH-K_1x03_P2.00mm_Horizontal -> Connector_JST:JST_PH_S3B-PH-SM4-TB_1x03-1MP_P2.00mm_Horizontal
Connections:
- net labels added: Relay6
- wire segments 248 -> 251
- no-connect marks 31 -> 28
Changed lines of the file:
@@
 F 0 "J12" H 6680 7442 50  0000 L CNN
 F 1 "Temp2" H 6680 7351 50  0000 L CNN
-F 2 "Connector_JST:JST_PH_S3B-PH-K_1x03_P2.00mm_Horizontal" H 6600 7400 50  0001 C CNN
+F 2 "Connector_JST:JST_PH_S3B-PH-SM4-TB_1x03-1MP_P2.00mm_Horizontal" H 6600 7400 50  0001 C CNN
 F 3 "https://www.jst-mfg.com/product/pdf/eng/ePH.pdf" H 6600 7400 50  0001 C CNN
 F 4 "JST Sales America Inc." H 6600 7400 50  0001 C CNN "Manufacturer"
@@
 F 0 "J9" H 6030 7442 50  0000 L CNN
 F 1 "Temp1" H 6030 7351 50  0000 L CNN
-F 2 "Connector_JST:JST_PH_S3B-PH-K_1x03_P2.00mm_Horizontal" H 5950 7400 50  0001 C CNN
+F 2 "Connector_JST:JST_PH_S3B-PH-SM4-TB_1x03-1MP_P2.00mm_Horizontal" H 5950 7400 50  0001 C CNN
 F 3 "https://www.jst-mfg.com/product/pdf/eng/ePH.pdf" H 5950 7400 50  0001 C CNN
 F 4 "JST Sales America Inc." H 5950 7400 50  0001 C CNN "Manufacturer"
@@
 	1    0    0    -1
 $EndComp
-Text Label 5350 7200 2    50   ~ 0
-Temp
 Text Notes 6450 7150 0    50   ~ 0
 Temperature
@@
 don't connect
 Text GLabel 6750 4350 0    50   Input ~ 0
-Relay1
+Relay5
 Text GLabel 6750 4250 0    50   Input ~ 0
-Relay2
+Relay4
 Text GLabel 6750 4150 0    50   Input ~ 0
 Relay3
 Text GLabel 6750 4050 0    50   Input ~ 0
-Relay4
+Relay2
 Text GLabel 6750 3950 0    50   Input ~ 0
-Relay5
+Relay1
 Text Notes 5100 600  0    50   ~ 0
 Power
@@
 F 0 "J6" H 4680 7342 50  0000 L CNN
 F 1 "Pressure" H 4680 7251 50  0000 L CNN
-F 2 "Connector_JST:JST_PH_S3B-PH-K_1x03_P2.00mm_Horizontal" H 4600 7300 50  0001 C CNN
+F 2 "Connector_JST:JST_PH_S3B-PH-SM4-TB_1x03-1MP_P2.00mm_Horizontal" H 4600 7300 50  0001 C CNN
 F 3 "https://www.jst-mfg.com/product/pdf/eng/ePH.pdf" H 4600 7300 50  0001 C CNN
 F 4 "JST Sales America Inc." H 4600 7300 50  0001 C CNN "Manufacturer"
@@
 NoConn ~ 7650 4550
 NoConn ~ 6850 4550
-NoConn ~ 6850 4450
 Text Notes 2450 5300 0    50   ~ 0
 Wifi (optional)
@@
 F 0 "J7" H 5322 6682 50  0000 R CNN
 F 1 "Acid Level" H 5450 6900 50  0000 R CNN
-F 2 "Connector_JST:JST_PH_S2B-PH-K_1x02_P2.00mm_Horizontal" H 5350 6800 50  0001 C CNN
+F 2 "Connector_JST:JST_PH_S2B-PH-SM4-TB_1x02-1MP_P2.00mm_Horizontal" H 5350 6800 50  0001 C CNN
 F 3 "https://www.jst-mfg.com/product/pdf/eng/ePH.pdf" H 5350 6800 50  0001 C CNN
 F 4 "JST Sales America Inc." H 5350 6800 50  0001 C CNN "Manufacturer"
@@
 F 0 "J10" H 6172 6682 50  0000 R CNN
 F 1 "Chlorine Level" H 6300 6900 50  0000 R CNN
-F 2 "Connector_JST:JST_PH_S2B-PH-K_1x02_P2.00mm_Horizontal" H 6200 6800 50  0001 C CNN
+F 2 "Connector_JST:JST_PH_S2B-PH-SM4-TB_1x02-1MP_P2.00mm_Horizontal" H 6200 6800 50  0001 C CNN
 F 3 "https://www.jst-mfg.com/product/pdf/eng/ePH.pdf" H 6200 6800 50  0001 C CNN
 F 4 "JST Sales America Inc." H 6200 6800 50  0001 C CNN "Manufacturer"
@@
 Probe_RST
 Text GLabel 950  2850 0    50   Input ~ 0
-Relay1
+Relay5
 Text GLabel 950  2950 0    50   Input ~ 0
-Relay2
+Relay4
 Text GLabel 950  3050 0    50   Input ~ 0
 Relay3
 Text GLabel 950  3150 0    50   Input ~ 0
-Relay4
+Relay2
 Text GLabel 950  3250 0    50   Input ~ 0
-Relay5
+Relay1
 Text GLabel 3350 3050 2    50   Input ~ 0
 ESP_TX
@@
 F 0 "J19" H 4772 5882 50  0000 R CNN
 F 1 "Flood sensor" H 5100 6150 50  0000 R CNN
-F 2 "Connector_JST:JST_PH_S3B-PH-K_1x03_P2.00mm_Horizontal" H 4800 5950 50  0001 C CNN
+F 2 "Connector_JST:JST_PH_S3B-PH-SM4-TB_1x03-1MP_P2.00mm_Horizontal" H 4800 5950 50  0001 C CNN
 F 3 "https://www.jst-mfg.com/product/pdf/eng/ePH.pdf" H 4800 5950 50  0001 C CNN
 F 4 "JST Sales America Inc." H 4800 5950 50  0001 C CNN "Manufacturer"
@@
 	0    1    1    0
 $EndComp
-NoConn ~ 3250 2650
-NoConn ~ 3250 2550
 $Comp
 L archive:Connector_Generic_Conn_02x07_Odd_Even J2
@@
 Wire Wire Line
 	7700 3950 7700 4550
+Text GLabel 3350 2550 2    50   Input ~ 0
+Relay6
+Wire Wire Line
+	3350 2550 3250 2550
+Text GLabel 6750 4450 0    50   Input ~ 0
+Relay6
+Wire Wire Line
+	6750 4450 6850 4450
+Text GLabel 5350 7200 0    50   Input ~ 0
+Temp
+Text GLabel 3350 2650 2    50   Input ~ 0
+Temp
+Wire Wire Line
+	3350 2650 3250 2650
 $EndSCHEMATC
