File: Controller/Controller.sch (KiCad schematic (older format))
At the start: 68 parts, among them IC1 LMP7715MF, J1 Probes, J10 Chlorine Level, J11 EXT_2, J12 Temp2, J13 Eth, J14 Acid Pump, J15 Chlorine Pump, J16 Filtration Pump, J17 Lighting, J18 Air, J19 Flood sensor, J2 Display, J20 EXT_I2C, J21 EXT_UART, J22 J1B1211CCD, J23 Relay_Ext, J3 ESP32, J4 EXT_SPI, J5 EXT_1, J6 Pressure, J7 Acid Level, J8 VInput, J9 Temp1, K1 ALQ305, K2 ALQ305, K3 ALQ305, K4 ALQ305, K5 ALQ305, K6 ALQ305, U1 Teensy4.1, U3 V7805-1000, U4 V7803-1000, U5 ULN2003A

Commit message: controller : - K7805M-1000R3 footprint - pressure use ads1014 - display connector position - air switch
Parts:
- removed C1: 100n, Capacitor_SMD:C_0805_2012Metric_Pad1.18x1.45mm_HandSolder, symbol archive:Device_C_Small
- removed IC1: LMP7715MF, SamacSys_Parts:SOT95P280X145-5N, symbol archive:SamacSys_Parts_LMP7715MF
- added C1: 1uF, Capacitor_SMD:C_0805_2012Metric_Pad1.18x1.45mm_HandSolder, symbol archive:Device_C
- added FB1, FB2: Ferrite_Bead_Small, Inductor_SMD:L_0805_2012Metric_Pad1.15x1.40mm_HandSolder, symbol archive:Device_Ferrite_Bead_Small
- added J24: air switch, Connector_JST:JST_PH_B3B-PH-K_1x03_P2.00mm_Vertical, symbol archive:Connector_Conn_01x03_Male
- added J25: EXT_3, Connector_JST:JST_PH_B5B-PH-K_1x05_P2.00mm_Vertical, symbol archive:Connector_Generic_Conn_01x05
- added JP1: Jumper_2_Open, Connector_PinHeader_2.54mm:PinHeader_1x02_P2.54mm_Vertical, symbol archive:Jumper_Jumper_2_Open
- added R4, R5: dnp, Resistor_SMD:R_0805_2012Metric_Pad1.20x1.40mm_HandSolder, symbol archive:Device_R_Small
- added R6, R7: 4K7, Resistor_SMD:R_0805_2012Metric_Pad1.20x1.40mm_HandSolder, symbol archive:Device_R_Small
- added U2: ADS1014IDGS, Package_SO:TSSOP-10_3x3mm_P0.5mm, symbol archive:Analog_ADC_ADS1014IDGS
- J1: footprint Connector_JST:JST_PH_B6B-PH-K_1x06_P2.00mm_Vertical -> Connector_JST:JST_PH_B5B-PH-K_1x05_P2.00mm_Vertical; symbol archive:Connector_Conn_01x06_Male -> archive:Connector_Generic_Conn_01x05
- J3: footprint Connector_PinSocket_2.54mm:PinSocket_2x03_P2.54mm_Vertical -> Connector_PinSocket_2.54mm:PinSocket_1x06_P2.54mm_Vertical
- R1: value 6.2k -> dnp
- R2: value 12k -> dnp
- U1: footprint teensy:Teensy41 -> lib_divers:Teensy41_nousb_noeth; symbol archive:teensy_Teensy4.1 -> archive:teensy41_nousb_noeth_Teensy41_nousb_noeth
- U3: value V7805-1000 -> K7805M-1000R3; footprint digikey-footprints:3-SIP_Module_V7805-1000 -> lib_divers:K7805M-1000R3; symbol archive:dk_DC-DC-Converters_V7805-1000 -> archive:K7805M-1000R3_K7805M-1000R3; Description DC DC CONVERTER 5V 5W -> (none); MANUFACTURER (none) -> Mornsun; MAXIMUM_PACKAGE_HEIGHT (none) -> 10.90 mm; Manufacturer CUI Inc. -> (none); PARTREV (none) -> 2020.01.08-A/5; STANDARD (none) -> Manufacturer Recommendations; digikey_pn 102-1715-ND -> (none); mpn V7805-1000 -> (none)
- U4: value V7803-1000 -> K7803M-1000R3; footprint digikey-footprints:3-SIP_Module_V7803-1000 -> lib_divers:K7803M-1000R3; symbol archive:dk_DC-DC-Converters_V7803-1000 -> archive:K7803M-1000R3_K7803M-1000R3; Description DC DC CONVERTER 3.3V 3.3W -> (none); MANUFACTURER (none) -> Mornsun; MAXIMUM_PACKAGE_HEIGHT (none) -> 10.9 mm; Manufacturer CUI Inc. -> (none); PARTREV (none) -> 2020.01.08-A/5; STANDARD (none) -> Manufacturer Recommendations; digikey_pn 102-1714-ND -> (none); mpn V7803-1000 -> (none)
Connections:
- net labels added: EXT_IO5, EXT_IO6, EXT_IO7, air_switch
- net labels removed: Pressure, Probe_RST
- wire segments 251 -> 284
- no-connect marks 28 -> 13
Other:
- note removed: "0-3.3V"
- note removed: "0-5V"
- moved on the sheet: C3, C4, C5, C6, C7, C8, F1, F2, J11, J20, J21, J4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

Commit message: increase Led resistor
Parts:
- R10, R11, R12, R13, R14, R3: value 180 -> 390
Changed lines of the file:
@@
 P 8700 2400
 F 0 "R14" H 8759 2446 50  0000 L CNN
-F 1 "180" H 8759 2355 50  0000 L CNN
+F 1 "390" H 8759 2355 50  0000 L CNN
 F 2 "Resistor_SMD:R_0805_2012Metric_Pad1.20x1.40mm_HandSolder" H 8700 2400 50  0001 C CNN
 F 3 "~" H 8700 2400 50  0001 C CNN
@@
 P 8450 2400
 F 0 "R13" H 8509 2446 50  0000 L CNN
-F 1 "180" H 8509 2355 50  0000 L CNN
+F 1 "390" H 8509 2355 50  0000 L CNN
 F 2 "Resistor_SMD:R_0805_2012Metric_Pad1.20x1.40mm_HandSolder" H 8450 2400 50  0001 C CNN
 F 3 "~" H 8450 2400 50  0001 C CNN
@@
 P 8250 2400
 F 0 "R12" H 8309 2446 50  0000 L CNN
-F 1 "180" H 8309 2355 50  0000 L CNN
+F 1 "390" H 8309 2355 50  0000 L CNN
 F 2 "Resistor_SMD:R_0805_2012Metric_Pad1.20x1.40mm_HandSolder" H 8250 2400 50  0001 C CNN
 F 3 "~" H 8250 2400 50  0001 C CNN
@@
 P 8050 2400
 F 0 "R11" H 8109 2446 50  0000 L CNN
-F 1 "180" H 8109 2355 50  0000 L CNN
+F 1 "390" H 8109 2355 50  0000 L CNN
 F 2 "Resistor_SMD:R_0805_2012Metric_Pad1.20x1.40mm_HandSolder" H 8050 2400 50  0001 C CNN
 F 3 "~" H 8050 2400 50  0001 C CNN
@@
 P 7850 2400
 F 0 "R10" H 7909 2446 50  0000 L CNN
-F 1 "180" H 7909 2355 50  0000 L CNN
+F 1 "390" H 7909 2355 50  0000 L CNN
 F 2 "Resistor_SMD:R_0805_2012Metric_Pad1.20x1.40mm_HandSolder" H 7850 2400 50  0001 C CNN
 F 3 "~" H 7850 2400 50  0001 C CNN
@@
 P 7700 2400
 F 0 "R3" H 7759 2446 50  0000 L CNN
-F 1 "180" H 7759 2355 50  0000 L CNN
+F 1 "390" H 7759 2355 50  0000 L CNN
 F 2 "Resistor_SMD:R_0805_2012Metric_Pad1.20x1.40mm_HandSolder" H 7700 2400 50  0001 C CNN
 F 3 "~" H 7700 2400 50  0001 C CNN
