File: Probe/Probe.sch (KiCad schematic (older format))
At the start: 52 parts, among them IC1 REF3440QDBVRQ1, IC2 LMP7721MAX_NOPB, IC3 ADM3260ARSZ-RL7, IC4 LMP7716MM_NOPB, IC5 MAX7321AEE+, J1 Interface, J2 Probe, J3 Addr, J5 Addr, J6 Interface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

Commit message: probe bom
Parts:
- IC1: Height 1.45 -> (none); Manufacturer (none) -> Texas Instruments; Manufacturer_Name Texas Instruments -> (none); Manufacturer_Part_Number REF3440QDBVRQ1 -> (none); Mouser Part Number 595-REF3440QDBVRQ1 -> (none); Mouser Price/Stock https://www.mouser.co.uk/ProductDetail/Texas-Instruments/RE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 -> (none); digikey_pn (none) -> 296-53237-1-ND; mouser_pn (none) -> 595-REF3440QDBVRQ1; mpn (none) -> REF3440QDBVRQ1
- IC2: Height 1.75 -> (none); Manufacturer (none) -> Texas Instruments; Manufacturer_Name Texas Instruments -> (none); Manufacturer_Part_Number LMP7721MAX/NOPB -> (none); Mouser Part Number 926-LMP7721MAX/NOPB -> (none); Mouser Price/Stock https://www.mouser.co.uk/ProductDetail/Texas-Instruments/LM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 -> (none); digikey_pn (none) -> LMP7721MAX/NOPB-ND; mouser_pn (none) -> 926-LMP7721MAX/NOPB; mpn (none) -> LMP7721MAX/NOPB
- IC3: Height 2 -> (none); Manufacturer (none) -> Analog Devices; Manufacturer_Name Analog Devices -> (none); Manufacturer_Part_Number ADM3260ARSZ-RL7 -> (none); Mouser Part Number 584-ADM3260ARSZ-RL7 -> (none); Mouser Price/Stock https://www.mouser.co.uk/ProductDetail/Analog-Devices/ADM32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 -> (none); digikey_pn (none) -> ADM3260ARSZ-RL7CT-ND; mouser_pn (none) -> 584-ADM3260ARSZ-RL7; mpn (none) -> ADM3260ARSZ-RL7
- IC4: Height 1.1 -> (none); Manufacturer (none) -> Texas Instruments; Manufacturer_Name Texas Instruments -> (none); Manufacturer_Part_Number LMP7716MM/NOPB -> (none); Mouser Part Number 926-LMP7716MM/NOPB -> (none); Mouser Price/Stock https://www.mouser.co.uk/ProductDetail/Texas-Instruments/LM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 -> (none); digikey_pn (none) -> LMP7716MME/NOPBCT-ND; mouser_pn (none) -> 926-LMP7716MM/NOPB; mpn (none) -> LMP7716MM/NOPB
- IC5: Height 1.75 -> (none); Manufacturer (none) -> Maxim Integrated; Manufacturer_Name Maxim Integrated -> (none); Manufacturer_Part_Number MAX7321AEE+ -> (none); Mouser Part Number 700-MAX7321AEE -> (none); Mouser Price/Stock https://www.mouser.co.uk/ProductDetail/Maxim-Integrated/MAX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 -> (none); digikey_pn (none) -> MAX7321AEE+-ND; farnell_pn (none) -> 2516740; mouser_pn (none) -> 700-MAX7321AEE; mpn (none) -> MAX7321AEE+
- J1, J6: Manufacturer (none) -> JST Sales America Inc.; digikey_pn (none) -> 455-1708-ND; farnell_pn (none) -> 9492453; mpn (none) -> B6B-PH-K-S
- J2: Description (none) -> BNC; Manufacturer (none) -> Amphenol RF; digikey_pn (none) -> ARF1690-ND; farnell_pn (none) -> 2293737; mouser_pn (none) -> 523-31-5431-10RFX; mpn (none) -> 031-5431-10RFX
- U1: Manufacturer (none) -> Texas Instruments; digikey_pn (none) -> 296-24932-1-ND; farnell_pn (none) -> 3004294; mouser_pn (none) -> 595-ADS1114IDGST
- U2: Manufacturer (none) -> Texas Instruments; digikey_pn (none) -> 296-39064-1-ND; farnell_pn (none) -> 3122292; mouser_pn (none) -> 595-LP5907MFX-4.5NPB
Changed lines of the file:
@@
 F 3 "https://componentsearchengine.com/Datasheets/1/ADM3260ARSZ-RL7.pdf" H 4600 1100 50  0001 L CNN
 F 4 "Digital Isolators Isolated I2C  & Power" H 4600 1000 50  0001 L CNN "Description"
-F 5 "2" H 4600 900 50  0001 L CNN "Height"
-F 6 "584-ADM3260ARSZ-RL7" H 4600 800 50  0001 L CNN "Mouser Part Number"
-F 7 "https://www.mouser.co.uk/ProductDetail/Analog-Devices/ADM3260ARSZ-RL7?qs=hpwIUhX6lWy5rzRvRSiwFQ%3D%3D" H 4600 700 50  0001 L CNN "Mouser Price/Stock"
-F 8 "Analog Devices" H 4600 600 50  0001 L CNN "Manufacturer_Name"
-F 9 "ADM3260ARSZ-RL7" H 4600 500 50  0001 L CNN "Manufacturer_Part_Number"
+F 5 "Analog Devices" H 4600 600 50  0001 L CNN "Manufacturer"
+F 6 "ADM3260ARSZ-RL7" H 4600 500 50  0001 L CNN "mpn"
+F 7 "584-ADM3260ARSZ-RL7" H 4600 800 50  0001 L CNN "mouser_pn"
+F 8 "ADM3260ARSZ-RL7CT-ND" H 3350 1100 50  0001 C CNN "digikey_pn"
+F 9 "" H 3350 1100 50  0001 C CNN "farnell_pn"
 	1    3350 1100
 	1    0    0    -1
@@
 F 1 "Interface" H 542 866 50  0000 C CNN
 F 2 "Connector_JST:JST_PH_B6B-PH-K_1x06_P2.00mm_Vertical" H 650 1300 50  0001 C CNN
-F 3 "~" H 650 1300 50  0001 C CNN
+F 3 "https://www.jst-mfg.com/product/pdf/eng/ePH.pdf" H 650 1300 50  0001 C CNN
+F 4 "JST Sales America Inc." H 650 1300 50  0001 C CNN "Manufacturer"
+F 5 "455-1708-ND" H 650 1300 50  0001 C CNN "digikey_pn"
+F 6 "9492453" H 650 1300 50  0001 C CNN "farnell_pn"
+F 7 "B6B-PH-K-S" H 650 1300 50  0001 C CNN "mpn"
 	1    650  1300
 	-1   0    0    -1
@@
 F 2 "Package_TO_SOT_SMD:SOT-23-5" H 6850 2350 50  0001 C CNN
 F 3 "http://www.ti.com/lit/ds/symlink/lp5907.pdf" H 6850 2500 50  0001 C CNN
+F 4 "Texas Instruments" H 6850 2000 50  0001 C CNN "Manufacturer"
+F 5 "296-39064-1-ND" H 6850 2000 50  0001 C CNN "digikey_pn"
+F 6 "3122292" H 6850 2000 50  0001 C CNN "farnell_pn"
+F 7 "595-LP5907MFX-4.5NPB" H 6850 2000 50  0001 C CNN "mouser_pn"
 	1    6850 2000
 	1    0    0    -1
@@
 F 3 "http://www.ti.com/lit/gpn/REF34-Q1" H 3250 4700 50  0001 L CNN
 F 4 "Automotive low-drift low-power small-footprint series voltage reference" H 3250 4600 50  0001 L CNN "Description"
-F 5 "1.45" H 3250 4500 50  0001 L CNN "Height"
-F 6 "595-REF3440QDBVRQ1" H 3250 4400 50  0001 L CNN "Mouser Part Number"
-F 7 "https://www.mouser.co.uk/ProductDetail/Texas-Instruments/REF3440QDBVRQ1?qs=byeeYqUIh0NTJm0mfXcM9Q%3D%3D" H 3250 4300 50  0001 L CNN "Mouser Price/Stock"
-F 8 "Texas Instruments" H 3250 4200 50  0001 L CNN "Manufacturer_Name"
-F 9 "REF3440QDBVRQ1" H 3250 4100 50  0001 L CNN "Manufacturer_Part_Number"
+F 5 "Texas Instruments" H 3250 4200 50  0001 L CNN "Manufacturer"
+F 6 "REF3440QDBVRQ1" H 3250 4100 50  0001 L CNN "mpn"
+F 7 "595-REF3440QDBVRQ1" H 3250 4400 50  0001 L CNN "mouser_pn"
+F 8 "296-53237-1-ND" H 2100 4700 50  0001 C CNN "digikey_pn"
 	1    2100 4700
 	1    0    0    1
@@
 F 3 "http://www.ti.com/lit/gpn/LMP7716" H 5650 4350 50  0001 L CNN
 F 4 "Dual Precision, 17 MHz, Low Noise, CMOS Input Amplifier" H 5650 4250 50  0001 L CNN "Description"
-F 5 "1.1" H 5650 4150 50  0001 L CNN "Height"
-F 6 "926-LMP7716MM/NOPB" H 5650 4050 50  0001 L CNN "Mouser Part Number"
-F 7 "https://www.mouser.co.uk/ProductDetail/Texas-Instruments/LMP7716MM-NOPB?qs=7lkVKPoqpbZs%2FD9QVWcbWA%3D%3D" H 5650 3950 50  0001 L CNN "Mouser Price/Stock"
-F 8 "Texas Instruments" H 5650 3850 50  0001 L CNN "Manufacturer_Name"
-F 9 "LMP7716MM/NOPB" H 5650 3750 50  0001 L CNN "Manufacturer_Part_Number"
+F 5 "926-LMP7716MM/NOPB" H 5650 4050 50  0001 L CNN "mouser_pn"
+F 6 "Texas Instruments" H 5650 3850 50  0001 L CNN "Manufacturer"
+F 7 "LMP7716MM/NOPB" H 5650 3750 50  0001 L CNN "mpn"
+F 8 "LMP7716MME/NOPBCT-ND" H 4600 4350 50  0001 C CNN "digikey_pn"
 	1    4600 4350
 	1    0    0    -1
@@
 F 3 "https://www.ti.com/general/docs/suppproductinfo.tsp?distId=10&gotoUrl=https%3A%2F%2Fwww.ti.com%2Flit%2Fgpn%2Flmp7721" H 3600 7050 50  0001 L CNN
 F 4 "Operational Amplifiers - Op Amps 3 Femtoampere Input Bias Current Precision Amplifier 8-SOIC -40 to 125" H 3600 6950 50  0001 L CNN "Description"
-F 5 "1.75" H 3600 6850 50  0001 L CNN "Height"
-F 6 "926-LMP7721MAX/NOPB" H 3600 6750 50  0001 L CNN "Mouser Part Number"
-F 7 "https://www.mouser.co.uk/ProductDetail/Texas-Instruments/LMP7721MAX-NOPB?qs=7lkVKPoqpbYZQwOlx%252BsPcg%3D%3D" H 3600 6650 50  0001 L CNN "Mouser Price/Stock"
-F 8 "Texas Instruments" H 3600 6550 50  0001 L CNN "Manufacturer_Name"
-F 9 "LMP7721MAX/NOPB" H 3600 6450 50  0001 L CNN "Manufacturer_Part_Number"
+F 5 "Texas Instruments" H 3600 6550 50  0001 L CNN "Manufacturer"
+F 6 "LMP7721MAX/NOPB" H 3600 6450 50  0001 L CNN "mpn"
+F 7 "926-LMP7721MAX/NOPB" H 3600 6750 50  0001 L CNN "mouser_pn"
+F 8 "LMP7721MAX/NOPB-ND" H 2550 7050 50  0001 C CNN "digikey_pn"
 	1    2550 7050
 	0    -1   -1   0
@@
 F 1 "Probe" H 1450 6573 50  0000 L CNN
 F 2 "Connector_Coaxial:BNC_Amphenol_B6252HB-NPP3G-50_Horizontal" H 1350 6600 50  0001 C CNN
-F 3 " ~" H 1350 6600 50  0001 C CNN
+F 3 "https://www.mouser.fr/datasheet/2/18/1/C31_5431_10rfx-2452641.pdf" H 1350 6600 50  0001 C CNN
+F 4 "BNC" H 1350 6600 50  0001 C CNN "Description"
+F 5 "Amphenol RF" H 1350 6600 50  0001 C CNN "Manufacturer"
+F 6 "	ARF1690-ND" H 1350 6600 50  0001 C CNN "digikey_pn"
+F 7 "031-5431-10RFX" H 1350 6600 50  0001 C CNN "mpn"
+F 8 "2293737" H 1350 6600 50  0001 C CNN "farnell_pn"
+F 9 "523-31-5431-10RFX" H 1350 6600 50  0001 C CNN "mouser_pn"
 	1    1350 6600
 	-1   0    0    1
@@
 F 2 "Package_SO:TSSOP-10_3x3mm_P0.5mm" H 5650 5400 50  0001 C CNN
 F 3 "http://www.ti.com/lit/ds/symlink/ads1113.pdf" H 5600 5000 50  0001 C CNN
+F 4 "Texas Instruments" H 5650 5900 50  0001 C CNN "Manufacturer"
+F 5 "296-24932-1-ND" H 5650 5900 50  0001 C CNN "digikey_pn"
+F 6 "3004294" H 5650 5900 50  0001 C CNN "farnell_pn"
+F 7 "595-ADS1114IDGST" H 5650 5900 50  0001 C CNN "mouser_pn"
 	1    5650 5900
 	1    0    0    -1
@@
 F 3 "https://componentsearchengine.com/Datasheets/2/MAX7321AEE+.pdf" H 2400 2900 50  0001 L CNN
 F 4 "Maxim MAX7321AEE+, 8-channel 8bit I/O Expander 400kHz, I2C, Serial, 16-Pin QSOP" H 2400 2800 50  0001 L CNN "Description"
-F 5 "1.75" H 2400 2700 50  0001 L CNN "Height"
-F 6 "700-MAX7321AEE" H 2400 2600 50  0001 L CNN "Mouser Part Number"
-F 7 "https://www.mouser.co.uk/ProductDetail/Maxim-Integrated/MAX7321AEE%2b?qs=LHmEVA8xxfYGcvkoPVuHog%3D%3D" H 2400 2500 50  0001 L CNN "Mouser Price/Stock"
-F 8 "Maxim Integrated" H 2400 2400 50  0001 L CNN "Manufacturer_Name"
-F 9 "MAX7321AEE+" H 2400 2300 50  0001 L CNN "Manufacturer_Part_Number"
+F 5 "700-MAX7321AEE" H 2400 2600 50  0001 L CNN "mouser_pn"
+F 6 "Maxim Integrated" H 2400 2400 50  0001 L CNN "Manufacturer"
+F 7 "MAX7321AEE+" H 2400 2300 50  0001 L CNN "mpn"
+F 8 "MAX7321AEE+-ND" H 1450 2900 50  0001 C CNN "digikey_pn"
+F 9 "2516740" H 1450 2900 50  0001 C CNN "farnell_pn"
 	1    1450 2900
 	1    0    0    -1
@@
 F 1 "Interface" H 1642 866 50  0000 C CNN
 F 2 "Connector_JST:JST_PH_B6B-PH-K_1x06_P2.00mm_Vertical" H 1750 1300 50  0001 C CNN
-F 3 "~" H 1750 1300 50  0001 C CNN
+F 3 "https://www.jst-mfg.com/product/pdf/eng/ePH.pdf" H 1750 1300 50  0001 C CNN
+F 4 "JST Sales America Inc." H 1750 1300 50  0001 C CNN "Manufacturer"
+F 5 "455-1708-ND" H 1750 1300 50  0001 C CNN "digikey_pn"
+F 6 "9492453" H 1750 1300 50  0001 C CNN "farnell_pn"
+F 7 "B6B-PH-K-S" H 1750 1300 50  0001 C CNN "mpn"
 	1    1750 1300
 	1    0    0    -1

Commit message: archive
Parts:
- C1, C15, C5: symbol Device:CP_Small -> archive:Device_CP_Small
- C10, C11, C12, C13, C14, C16, C17, C18, C2, C3, C4, C6, C7, C8, C9: symbol Device:C_Small -> archive:Device_C_Small
- D1, D2: symbol Device:LED -> archive:Device_LED
- IC1: symbol SamacSys_Parts:REF3440QDBVRQ1 -> archive:SamacSys_Parts_REF3440QDBVRQ1
- IC2: symbol SamacSys_Parts:LMP7721MAX_NOPB -> archive:SamacSys_Parts_LMP7721MAX_NOPB
- IC3: symbol SamacSys_Parts:ADM3260ARSZ-RL7 -> archive:SamacSys_Parts_ADM3260ARSZ-RL7
- IC4: symbol SamacSys_Parts:LMP7716MM_NOPB -> archive:SamacSys_Parts_LMP7716MM_NOPB
- IC5: symbol max7321aee:max7321aee+ -> archive:max7321aee_max7321aee+
- J1, J6: symbol Connector:Conn_01x06_Female -> archive:Connector_Conn_01x06_Female
- J2: symbol Connector:Conn_Coaxial -> archive:Connector_Conn_Coaxial
- J3, J5: symbol Connector_Generic:Conn_02x04_Odd_Even -> archive:Connector_Generic_Conn_02x04_Odd_Even
- R1, R10, R11, R12, R13, R14, R15, R16, R17, R18, R19, R2, R20, R3, R4, R5, R6, R7, R8, R9: symbol Device:R_Small -> archive:Device_R_Small
- U1: symbol Analog_ADC:ADS1114IDGS -> archive:Analog_ADC_ADS1114IDGS
- U2: symbol Regulator_Linear:LP5907MFX-4.5 -> archive:Regulator_Linear_LP5907MFX-4.5
