File: display/display.sch (KiCad schematic (older format))
At the start: 2 parts, among them J1 MCU, J2 Disp

Commit message: display
Parts:
- J1: symbol Connector_Generic:Conn_02x07_Odd_Even -> archive:Connector_Generic_Conn_02x07_Odd_Even
- J2: symbol Connector_Generic:Conn_02x20_Odd_Even -> archive:Connector_Generic_Conn_02x20_Odd_Even
Changed lines of the file:
@@
 $EndDescr
 $Comp
-L Connector_Generic:Conn_02x20_Odd_Even J2
+L archive:Connector_Generic_Conn_02x20_Odd_Even J2
 U 1 1 62095E19
 P 3750 1650
@@
 $EndComp
 $Comp
-L Connector_Generic:Conn_02x07_Odd_Even J1
+L archive:Connector_Generic_Conn_02x07_Odd_Even J1
 U 1 1 6209B0F5
 P 1600 1400
@@
 LCD_MOSI
 $Comp
-L power:GND #PWR01
+L archive:power_GND #PWR01
 U 1 1 620A2A3D
 P 1250 1100
@@
 NoConn ~ 1900 1100
 $Comp
-L power:+3V3 #PWR02
+L archive:power_+3V3 #PWR02
 U 1 1 620A46C2
 P 2050 1200
@@
 	1900 1200 2050 1200
 $Comp
-L power:GND #PWR03
+L archive:power_GND #PWR03
 U 1 1 620A53DF
 P 3450 750
@@
 $EndComp
 $Comp
-L power:+3V3 #PWR04
+L archive:power_+3V3 #PWR04
 U 1 1 620A6063
 P 4150 750
@@
 Text GLabel 4150 2050 2    50   Input ~ 0
 LCD_MISO
-Text GLabel 4150 1850 2    50   Input ~ 0
-LCD_SCLK
 Text GLabel 3450 1950 0    50   Input ~ 0
 LCD_DC
@@
 Wire Wire Line
 	4150 2050 4050 2050
-Wire Wire Line
-	4050 1850 4150 1850
 Wire Wire Line
 	4050 750  4150 750
@@
 NoConn ~ 4050 2650
 $Comp
-L power:PWR_FLAG #FLG0101
+L archive:power_PWR_FLAG #FLG0101
 U 1 1 620B59E8
 P 2050 1000
@@
 $EndComp
 $Comp
-L power:PWR_FLAG #FLG0102
+L archive:power_PWR_FLAG #FLG0102
 U 1 1 620B642E
 P 1300 1000
@@
 	2050 1000 2050 1200
 Connection ~ 2050 1200
+Wire Wire Line
+	4050 1850 4150 1850
+Text GLabel 4150 1850 2    50   Input ~ 0
+LCD_SCLK
 $EndSCHEMATC
